File: prj3-datalogger.kicad_sch (KiCad schematic)
At the start: 25 parts, among them U1 24LC1025, U2 24LC1025, U3 DS1337S_, U4 ATMEGA328P-AU, Y1 32.768 KHz, Y2 16 MHz

Commit message: added comments
Other:
- note added: "EEPROM (memory)"
- note added: "MCU"
- note added: "Mounting holes"
- note added: "Real time clock"
- moved on the sheet: BT1, C1, C2, C3, C4, C5, D1, D2, H1, H2, H3, H4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

Commit message: text amends and Vcc label at batt schem
Connections:
- net VCC: now also BT1.1 (+), C5.1, D1.2 (A), U4.18 (AVCC), U4.4 (VCC)
Changed lines of the file:
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@@
-	(wire
-		(pts
-			(xy 256.54 29.21) (xy 267.97 29.21)
-		)
-		(stroke
-			(width 0)
-			(type default)
-		)
-	)
 	(wire
 		(pts
@@
 	(wire
 		(pts
-			(xy 247.65 29.21) (xy 256.54 29.21)
+			(xy 247.65 29.21) (xy 267.97 29.21)
 		)
 		(stroke
@@
 		(effects
 			(font
+				(size 1.27 1.27)
+			)
+			(justify left bottom)
+		)
+	)
+	(label "VCC"
+		(at 262.89 29.21 0)
+		(effects
+			(font

Commit message: Fixed defects in schematic
Connections:
- net SCL: no longer D2.2 (A), U4.17 (PB5)
- new net SCK: D2.2 (A), U4.17 (PB5)
Other:
- sheet connectors ports: added SCK; removed none
Changed lines of the file:
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@@
 	(wire
 		(pts
-			(xy 83.82 139.7) (xy 83.82 146.05)
-		)
-		(stroke
-			(width 0)
-			(type default)
-		)
-	)
-	(wire
-		(pts
 			(xy 229.87 72.39) (xy 234.95 72.39)
 		)
@@
 		)
 	)
-	(label "SCL"
+	(label "SCK"
 		(at 199.39 49.53 180)
 		(effects
@@
 		)
 	)
+	(label "SCK"
+		(at 201.93 156.21 0)
+		(effects
+			(font
+				(size 1.27 1.27)
+			)
+			(justify left bottom)
+		)
+	)
 	(label "VCC"
 		(at 38.1 151.13 180)
@@
 	)
 	(symbol
-		(lib_id "power:PWR_FLAG")
-		(at 83.82 139.7 0)
-		(unit 1)
-		(body_style 1)
-		(exclude_from_sim no)
-		(in_bom yes)
-		(on_board yes)
-		(in_pos_files yes)
-		(dnp no)
-		(fields_autoplaced yes)
-		(property "Reference" "#FLG03"
-			(at 83.82 137.795 0)
-			(hide yes)
-			(show_name no)
-			(do_not_autoplace no)
-			(effects
-				(font
-					(size 1.27 1.27)
-				)
-			)
-		)
-		(property "Value" "PWR_FLAG"
-			(at 83.82 134.62 0)
-			(show_name no)
-			(do_not_autoplace no)
-			(effects
-				(font
-					(size 1.27 1.27)
-				)
-			)
-		)
-		(property "Footprint" ""
-			(at 83.82 139.7 0)
-			(hide yes)
-			(show_name no)
-			(do_not_autoplace no)
-			(effects
-				(font
-					(size 1.27 1.27)
-				)
-			)
-		)
-		(property "Datasheet" ""
-			(at 83.82 139.7 0)
-			(hide yes)
-			(show_name no)
-			(do_not_autoplace no)
-			(effects
-				(font
-					(size 1.27 1.27)
-				)
-			)
-		)
-		(property "Description" "Special symbol for telling ERC where power comes from"
-			(at 83.82 139.7 0)
-			(hide yes)
-			(show_name no)
-			(do_not_autoplace no)
-			(effects
-				(font
-					(size 1.27 1.27)
-				)
-			)
-		)
-		(pin "1"
-		)
-		(instances
-			(project "prj3-datalogger"
-				(path "/6e9d2065-7b61-4fa9-8ffc-cd31ce5c40e2"
-					(reference "#FLG03")
-					(unit 1)
-				)
-			)
-		)
-	)
-	(symbol
 		(lib_id "Device:LED")
 		(at 177.8 34.29 0)
@@
 			(effects
 				(font
+					(size 1.27 1.27)
+				)
+				(justify right)
+			)
+		)
+		(pin "SCK" passive
+			(at 201.93 156.21 0)
+			(effects
+				(font
