File: prj3-datalogger.kicad_pcb (KiCad board)
At the start: 2 copper layers, 56 x 33 mm, 29 parts, among them J1 Conn_01x04_Pin, J2 Conn_01x04_Pin, J3 Conn_01x09_Pin, J4 Conn_02x03_Odd_Even, U1 24LC1025, U2 24LC1025, U3 DS1337S_, U4 ATMEGA328P-AU, Y1 32.768 KHz, Y2 16 MHz

Commit message: Fixed 2layer PCB
Connections:
- BT1 pad 1: Net-(BT1-+) -> /VCC
- C5 pad 1: Net-(BT1-+) -> /VCC
- D1 pad 2: Net-(BT1-+) -> /VCC
- D2 pad 2: /SCL -> /SCK
- J4 pad 3: /SCL -> /SCK
- U4 pad 17: /SCL -> /SCK
- U4 pad 18: Net-(BT1-+) -> /VCC
- U4 pad 4: Net-(BT1-+) -> /VCC
Routing:
- net /SCK: track 0.00 -> 80.3 mm, vias 0 -> 3
- net /VCC: track 152.1 -> 189.5 mm, vias 9 -> 13
- net Net-(BT1-+): track 35.8 -> 0.00 mm, vias 2 -> 0
- net /SCL: track 113.9 -> 82.6 mm
- net /RESET: track 33.3 -> 39.5 mm
- net /SDA: track 119.1 -> 120.9 mm
