File: prj3-datalogger.kicad_pcb (KiCad board)
At the start: 4 copper layers, 56 x 33 mm, 30 parts, among them J1 Conn_01x04_Pin, J2 Conn_01x04_Pin, J3 Conn_01x09_Pin, J4 Conn_02x03_Odd_Even, U1 24LC1025, U2 24LC1025, U3 DS1337S_, U4 ATMEGA328P-AU, Y1 32.768 KHz, Y2 16 MHz

Commit message: Fixed 4layer PCB
Connections:
- BT1 pad 1: Net-(BT1-+) -> /VCC
- C5 pad 1: Net-(BT1-+) -> /VCC
- D1 pad 2: Net-(BT1-+) -> /VCC
- D2 pad 2: /SCL -> /SCK
- J4 pad 3: /SCL -> /SCK
- U4 pad 17: /SCL -> /SCK
- U4 pad 18: Net-(BT1-+) -> /VCC
- U4 pad 4: Net-(BT1-+) -> /VCC
Routing:
- net /SCK: track 0.00 -> 61.2 mm, vias 0 -> 2
- net Net-(BT1-+): track 39.5 -> 0.00 mm, vias 3 -> 0
- net /VCC: track 42.1 -> 65.9 mm, vias 7 -> 10
- net /SCL: track 115.2 -> 98.6 mm, vias 8 -> 5
- net /MISO: track 29.8 -> 28.4 mm
- net Net-(U4-PB7): track 42.7 -> 43.5 mm, vias 4 -> 5
- net GND: track 34.6 -> 33.9 mm
